Commit message: Nav stack working!

File: catkin_ws/src/robot_description/urdf/robot_description.urdf (robot description, URDF)
Before this commit: robot robot_description, 2 links, 1 joints
Links:
- added link laser_link; visual box size=0.08 0.08 0.1
Joints:
- added joint laser_joint: type fixed, parent base_link, child laser_link, origin xyz=-0.33 -0.35 0.3 rpy=0 0 0

Commit message: Files update

File: catkin_ws/src/robot_description/urdf/robot_description.urdf (robot description, URDF)
Before this commit: robot robot_description, 3 links, 2 joints
Links:
- removed link base_all
- added link laser; visual box size=0.1 0.04 0.2
- link base_link: geometry collision mesh filename=package://robot_description/meshes/base_link.STL; visual mesh filename=package://robot_description/meshes/base_all.STL
Joints:
- removed joint all
- added joint lidar_joint: type fixed, parent laser_link, child laser, origin xyz=0 0 0 rpy=0 0 3.14159
- joint laser_joint: origin xyz=-0.33 -0.35 0.3 rpy=0 0 0 -> xyz=0.19 0.01 0.20 rpy=0 0 0
